File: nzxt-gamma-usb3.brd (EAGLE design)
At the start: 94 x 21 mm, 8 parts, among them J1 SJ1-3545N, J2 SJ1-3545N, J3 GSB311131HR, J4 GSB311131HR

Commit message: Named some nets for debug, added some schematic detail
Connections:
- net N$1 renamed SENSE_1_RET
- net N$3 renamed SENSE1_1_SEND
- net N$4 renamed P_1_R
- net N$5 renamed P_2_L
- net N$6 renamed SENSE_2_RET
- net N$8 renamed P_2_R
Changed lines of the file:
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@@
 </autorouter>
 <elements>
-<element name="J1" library="dylans-parts" library_urn="urn:adsk.eagle:library:6331967" package="CUI_SJ1-3545N" package3d_urn="urn:adsk.eagle:package:6331970/2" value="SJ1-3545N" x="85" y="18" smashed="yes" rot="R270">
+<element name="J1" library="dylans-parts" library_urn="urn:adsk.eagle:library:6331967" package="CUI_SJ1-3545N" package3d_urn="urn:adsk.eagle:package:6331970/3" value="SJ1-3545N" x="85" y="18" smashed="yes" rot="R270">
 <attribute name="MANUFACTURER" value="CUI" x="85" y="18" size="1.778" layer="27" rot="R270" display="off"/>
 <attribute name="NAME" x="78.725" y="9.098" size="1.781309375" layer="25" font="vector" rot="SR0" align="top-left"/>
@@
 <attribute name="VALUE" x="77.87246875" y="20.87968125" size="1.78213125" layer="27" font="vector" rot="R270" align="top-left"/>
 </element>
-<element name="J2" library="dylans-parts" library_urn="urn:adsk.eagle:library:6331967" package="CUI_SJ1-3545N" package3d_urn="urn:adsk.eagle:package:6331970/2" value="SJ1-3545N" x="71" y="18" smashed="yes" rot="R270">
+<element name="J2" library="dylans-parts" library_urn="urn:adsk.eagle:library:6331967" package="CUI_SJ1-3545N" package3d_urn="urn:adsk.eagle:package:6331970/3" value="SJ1-3545N" x="71" y="18" smashed="yes" rot="R270">
 <attribute name="MANUFACTURER" value="CUI" x="71" y="18" size="1.778" layer="27" rot="R270" display="off"/>
 <attribute name="NAME" x="64.725" y="9.098" size="1.781309375" layer="25" font="vector" rot="SR0" align="top-left"/>
@@
 </polygon>
 </signal>
-<signal name="N$1">
+<signal name="SENSE_1_RET">
 <contactref element="JP1" pad="10"/>
 <contactref element="J2" pad="4"/>
@@
 <wire x1="68.58" y1="8.255" x2="66" y2="10.835" width="0.254" layer="1"/>
 </signal>
-<signal name="N$5">
+<signal name="P_2_L">
 <contactref element="J1" pad="2"/>
 <contactref element="JP1" pad="3"/>
@@
 <wire x1="85.09" y1="6.985" x2="81.28" y2="10.795" width="0.254" layer="1"/>
 </signal>
-<signal name="N$6">
+<signal name="SENSE_2_RET">
 <contactref element="JP1" pad="1"/>
 <contactref element="J1" pad="4"/>
@@
 <wire x1="85.725" y1="7.62" x2="82.5" y2="10.845" width="0.254" layer="1"/>
 </signal>
-<signal name="N$4">
+<signal name="P_1_R">
 <contactref element="JP1" pad="7"/>
 <contactref element="J2" pad="3"/>
@@
 <wire x1="74.93" y1="9.525" x2="73.5" y2="10.955" width="0.254" layer="1"/>
 </signal>
-<signal name="N$3">
+<signal name="SENSE1_1_SEND">
 <contactref element="JP1" pad="2"/>
 <contactref element="J1" pad="5"/>
@@
 <wire x1="85.09" y1="5.08" x2="87.5" y2="7.49" width="0.254" layer="16"/>
 </signal>
-<signal name="N$8">
+<signal name="P_2_R">
 <contactref element="JP1" pad="4"/>
 <contactref element="J1" pad="3"/>
